File: Signal_Controller.sch (KiCad schematic (older format))
At the start: 2 parts

Commit message: Schematic just about finished
Parts:
- added C? (x5): 1uF, symbol C
- added C? (x2): 18pF, symbol C
- added C?: 10uF, symbol C
- added C?: 0.1uF, symbol C
- added D? (x3): LED, symbol LED
- added J?: BARREL_JACK, symbol BARREL_JACK
- added J?: CONN_02X03, symbol CONN_02X03
- added J?: CONN_01X03, symbol CONN_01X05
- added Q? (x3): 2N7002P,215, symbol 2N7002P,215
- added R? (x6): R, symbol R
- added R?: 10K, symbol R
- added R? (x2): 22, symbol R
- added RL? (x3): G5LE-1, symbol G5LE-1
- added SW?: SW_Push, symbol SW_Push
- added U?: AZ1117IH-5.0TRG1, symbol AZ1117IH-5.0TRG1
- added Y?: Crystal, symbol Crystal
Connections:
- net GND: now also U?.33 ((~HWB~)PE2), U?.5 (UGND), C?.1, C?.1, C?.2, C?.2, C?.2, C?.2, C?.2, C?.2, C?.2, D?.1 (K), D?.1 (K), D?.1 (K), J?.1 (P1), J?.2, J?.3, J?.6 (P6), Q?.3 (D), Q?.3 (D), Q?.3 (D), R?.2, R?.2, R?.2, RL?.4, RL?.4, RL?.4, SW?.2, U?.1 (GND)
- net MOSI: now reaches U?.10 ((PDI/MOSI/PCINT2)PB2)
- net MOSI: now also J?.4 (P4)
- net MISO: now reaches U?.11 ((PDO/MISO/PCINT3)PB3)
- net MISO: now also J?.1 (P1)
- net RST: now reaches U?.13 (RESET)
- net RST: now also J?.5 (P5), R?.2, SW?.1
- net +5V: now reaches U?.14 (VCC)
- net +5V: now also U?.2 (UVCC), U?.24 (AVCC), U?.34 (VCC), U?.44 (AVCC), C?.1, C?.1, C?.1, J?.2 (P2), R?.1, R?.1, U?.2 (VO)
- net at U?.16 (XTAL2): now also C?.2, Y?.2
- net at U?.17 (XTAL1): now also C?.2, Y?.1
- net at U?.22 ((XCK1/~CTS~)PD5): now also R?.2
- net RELAY_1: now reaches U?.25 ((ICP2/ADC8)PD4)
- net RELAY_1: now also Q?.1 (G), R?.1
- net RELAY_2: now reaches U?.26 ((T1/~OC4D~/ADC9)PD6)
- net RELAY_2: now also Q?.1 (G), R?.1
- net RELAY_3: now reaches U?.27 ((T0/OC4D/ADC10)PD7)
- net RELAY_3: now also Q?.1 (G), R?.1
- net RELAY_4: now reaches U?.28 ((ADC11/PCINT4)PB4)
- net RELAY_4: now also J?.4 (P4)
- net RELAY_5: now reaches U?.29 ((ADC12/OC1A/~OC4B~/PCINT12)PB5)
- net RELAY_5: now also J?.3 (P3)
- net at U?.3 (D-): now also R?.1
- net RELAY_6: now reaches U?.30 ((ADC13/OC1B/OC4B/PCINT13)PB6)
- net RELAY_6: now also J?.2 (P2)
- net at U?.4 (D+): now also R?.1
- net at U?.42 (AREF): now also C?.1
- net at U?.6 (UCAP): now also C?.1
- net V_BUS: now reaches U?.7 (VBUS)
- net V_BUS: now also J?.1 (VBUS), C?.1
- net SCK: now reaches U?.9 ((SCLK/PCINT1)PB1)
- net SCK: now also J?.3 (P3)
- net D-: now reaches J?.2 (D-)
- net D-: now also R?.2
- net D+: now reaches J?.3 (D+)
- net D+: now also R?.2
- new net: D?.2 (A), R?.2
- new net: D?.2 (A), R?.1 (x2)
- new net: Q?.2 (S), RL?.5 (x3)
- new net +12V: C?.1, J?.1, J?.5 (P5), RL?.3, RL?.3, RL?.3, U?.3 (VI)
- new net BULB: RL?.1
- new net COIL_1A: RL?.1, RL?.1
- no-connect marks 0 -> 1
Other:
- note added: "ICSP Header"
- note added: "MCU/Peripheral Power"
- note added: "Output Relays"
- note added: "Power Input"
- note added: "Relay Expansion Board"
- note added: "USB Input (Programming)"
- moved on the sheet: J?, U?

Commit message: assigning footprints/generating netlist
Parts:
- gave numbers to parts that had none: 35
