File: Signal_Controller_MCU_Board/_saved_Signal_Controller.sch (KiCad schematic (older format))
At the start: 50 parts, among them J1 BARREL_JACK, J2 USB_OTG, J3 CONN_02X03, J4 CONN_01X03, J5 CONN_01X02, J6 CONN_01X02, J7 CONN_01X02, J8 CONN_01X07, Q1 2N7002P,215, Q2 2N7002P,215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

Commit message: First pass of PCB finished
Parts:
- C7, C8: value 18pF -> 22pF
- Y1: footprint (none) -> Crystals:Crystal_SMD_3225-4pin_3.2x2.5mm
Connections:
- net COIL_1A: now also J5.1 (P1); no longer J5.2 (P2)
- net COIL_1B: now also J5.2 (P2); no longer J5.1 (P1)
Changed lines of the file:
@@
 F 0 "Y1" H 4100 5050 50  0000 C CNN
 F 1 "Crystal" V 3950 5050 50  0000 C CNN
-F 2 "" H 4100 4900 50  0001 C CNN
+F 2 "Crystals:Crystal_SMD_3225-4pin_3.2x2.5mm" H 4100 4900 50  0001 C CNN
 F 3 "" H 4100 4900 50  0001 C CNN
 	1    4100 4900
@@
 P 3850 4700
 F 0 "C7" V 3800 4550 50  0000 L CNN
-F 1 "18pF" V 3900 4450 50  0000 L CNN
+F 1 "22pF" V 3900 4450 50  0000 L CNN
 F 2 "Capacitors_SMD:C_0603" H 3888 4550 50  0001 C CNN
 F 3 "" H 3850 4700 50  0001 C CNN
@@
 P 3850 5100
 F 0 "C8" V 3900 4950 50  0000 L CNN
-F 1 "18pF" V 3800 4850 50  0000 L CNN
+F 1 "22pF" V 3800 4850 50  0000 L CNN
 F 2 "Capacitors_SMD:C_0603" H 3888 4950 50  0001 C CNN
 F 3 "" H 3850 5100 50  0001 C CNN
@@
 Text Notes 650  850  0    60   ~ 0
 Barrel or Terminal Block
+Text HLabel 1400 4750 2    60   Input ~ 0
+COIL_1A
 Text HLabel 1400 4650 2    60   Input ~ 0
-COIL_1A
-Text HLabel 1400 4750 2    60   Input ~ 0
 COIL_1B
 Text HLabel 1400 5150 2    60   Input ~ 0
